File: schematics/eggbothat.brd (EAGLE design)
At the start: 100 x 80 mm, 29 parts

Commit message: schematic fixes
Parts:
- C1: device rcl:E5-10,5 -> rcl:E2,5-5
- R10, R11, R12, R2, R3, R4, R5, R6, R7, R8, R9: device rcl:R0402 -> rcl:R1206
- moved R2 10.9 mm to (53.3, 41.5)
- moved C1 2.68 mm to (14.0, 42.8)
- moved R3 1.80 mm to (30.5, 41.9)
- moved R8 1.53 mm to (15.2, 51.6)
- moved R4 1.34 mm to (27.9, 19.9)
- moved R9 1.27 mm to (15.2, 48.3)
- moved R5 1.27 mm to (20.7, 20.7)
- moved R12 1.27 mm to (45.7, 43.2)
- moved 12VOLT 0.95 mm to (72.0, 28.8)
- moved R6 0.95 mm to (71.5, 19.1)
- moved R11 0.85 mm to (66.0, 41.1)
- moved R10 0.42 mm to (10.2, 37.7), turned to 270 degrees
Routing:
- net GND: track 377.8 -> 332.6 mm, vias 2 -> 0
- net VCC: track 262.9 -> 250.6 mm
- net +3V3: track 209.5 -> 198.6 mm, vias 0 -> 1
- net N$10: track 6.13 -> 13.5 mm
- net N$20: track 26.7 -> 27.8 mm
- net MTX6: track 34.2 -> 33.1 mm
- net N$13: track 12.6 -> 13.5 mm
- net +12V: track 36.5 -> 35.6 mm
- net MTX8: track 34.1 -> 33.3 mm
- net I2C_SDA: track 17.4 -> 18.0 mm
- net I2C2_SDA: track 24.8 -> 25.3 mm
- net N$17: track 3.73 -> 3.17 mm

Commit message: try pen motor elevator
Parts:
- moved SERVO1 30.8 mm to (4.23, 9.31), turned to 270 degrees
- moved SERVO2 25.4 mm to (4.23, 18.6), turned to 90 degrees
- moved 12VOLT 3.39 mm to (75.4, 28.8)
- moved R6 3.39 mm to (74.9, 19.1)
- moved U$1 3.39 mm to (68.2, 34.3)
- moved DIVPEN 3.39 mm to (64.3, 40.6)
- moved NUMPAD 3.39 mm to (64.3, 15.7)
- moved R12 3.39 mm to (49.1, 43.2)
- moved R5 3.39 mm to (24.1, 20.7)
- moved RASPBERRY 3.39 mm to (40.2, 53.3)
- moved STEPPER_EGG 3.39 mm to (37.7, 28.4)
- moved STEPPER_PEN 3.39 mm to (60.5, 28.4)
- moved U$2 3.39 mm to (45.3, 34.3)
- moved C1 3.39 mm to (17.4, 42.8)
- moved R10 3.39 mm to (13.5, 37.7)
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Routing:
- net PWM2: track 5.93 -> 46.5 mm
- net PWM1: track 4.32 -> 41.1 mm
- net VCC: track 250.6 -> 214.5 mm
- net GND: track 332.6 -> 308.1 mm
- net SPI_MOSI: track 49.8 -> 45.3 mm
