File: schematics/eggbothat3.sch (EAGLE design)
At the start: 43 parts

Commit message: versions 2,3 of electronics
Parts:
- removed ENDSTOPS: (no value), con-lstb:MA03-2
- removed OLED2: (no value), con-lstb:MA04-1
- removed R8, R9: 4k7, rcl:R-EU_R1206
- removed RASPBERRY: RPI-B-V2SHIELD, levelshifter:RPI-B-V2SHIELD
- removed SHIFTER1: LEVELSHIFTER, levelshifter:LEVELSHIFTER
- added EP1, EP2: (no value), con-lstb:MA03-1
Connections:
- removed net +3V3: ENDSTOPS.5, ENDSTOPS.6, OLED2.1, R8.2, R9.2, RASPBERRY.+3V3, SHIFTER1.VCCA
- removed net I2C2_SCL: OLED2.3, R9.1, RASPBERRY.GPIO3/I2C1_SCL
- removed net I2C2_SDA: OLED2.4, R8.1, RASPBERRY.GPIO2/I2C1_SDA
- removed net SPI33_CLK: RASPBERRY.GPIO11/SPI0_SLCK, SHIFTER1.A3
- removed net SPI33_CS1: RASPBERRY.GPIO8/SPI0_CE0, SHIFTER1.A2
- removed net SPI33_MISO: RASPBERRY.GPIO9/SPI0_MISO, SHIFTER1.A4
- removed net SPI33_MOSI: RASPBERRY.GPIO10/SPI0_MOSI, SHIFTER1.A5
- removed net SPI_CLK: SHIFTER1.B3, U$4.D13
- removed net SPI_CS1: SHIFTER1.B2, U$4.D10
- removed net SPI_MISO: SHIFTER1.B4, U$4.D12
- removed net SPI_MOSI: SHIFTER1.B5, U$4.D11
- new net LED-INTERN: U$4.D13
- new net NC1: U$4.D12
- net E-DIR: now also U$4.D2; no longer U$4.D3
- net E-STEP: now also U$4.D3; no longer U$4.D2
- net END1: now also EP1.2, U$4.D8; no longer ENDSTOPS.4, RASPBERRY.UART0_TXD/GPIO14
- net END2: now also EP2.2, U$4.D9; no longer ENDSTOPS.3, RASPBERRY.UART0_RXD/GPIO15
- net GND: now also EP1.1, EP2.1; no longer ENDSTOPS.1, ENDSTOPS.2, OLED2.2, RASPBERRY.GND, SHIFTER1.GND
- net P-DIR: now also U$4.D5; no longer U$4.D7
- net P-EN: now also U$4.D7; no longer U$4.D9
- net P-STEP: now also U$4.D6; no longer U$4.D8
- net PWM1: now also U$4.D10; no longer U$4.D5
- net PWM2: now also U$4.D11; no longer U$4.D6
- net VCC: now also EP1.3, EP2.3; no longer RASPBERRY.+5V, SHIFTER1.VCCB
Other:
- note removed: "TODO: Check Rasopi ground"
